File: PCBs/logic/logic.kicad_sch (KiCad schematic)
At the start: 10 parts, among them J1 PWR_Conn, J2 Conn_01x04, SW1 next_Button, U8 ESP32-C6-DEVKITC-1-N8

Commit message: Logic PCB finished
Parts:
- R1: value R -> 10k; footprint (none) -> Resistor_THT:R_Axial_DIN0207_L6.3mm_D2.5mm_P10.16mm_Horizontal
- RV1: footprint (none) -> Connector_PinHeader_2.54mm:PinHeader_1x03_P2.54mm_Vertical
- SW1: footprint (none) -> Connector_PinHeader_2.54mm:PinHeader_1x02_P2.54mm_Vertical
Connections:
- net +3.3V: now also RV1.3; no longer RV1.1
- net GND: now also RV1.1; no longer RV1.3
- no-connect marks 1 -> 20
Other:
- moved on the sheet: RV1
Changed lines of the file:
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@@
 		(color 0 0 0 0)
+	)
+	(junction
+		(at 125.73 44.45)
+		(diameter 0)
+		(color 0 0 0 0)
+	)
+	(junction
+		(at 125.73 46.99)
+		(diameter 0)
+		(color 0 0 0 0)
+	)
+	(no_connect
+		(at 72.39 125.73)
+	)
+	(no_connect
+		(at 113.03 110.49)
 	)
 	(no_connect
 		(at 72.39 102.87)
 	)
+	(no_connect
+		(at 72.39 128.27)
+	)
+	(no_connect
+		(at 113.03 123.19)
+	)
+	(no_connect
+		(at 113.03 107.95)
+	)
+	(no_connect
+		(at 72.39 120.65)
+	)
+	(no_connect
+		(at 113.03 118.11)
+	)
+	(no_connect
+		(at 113.03 125.73)
+	)
+	(no_connect
+		(at 72.39 105.41)
+	)
+	(no_connect
+		(at 113.03 102.87)
+	)
+	(no_connect
+		(at 113.03 130.81)
+	)
+	(no_connect
+		(at 72.39 113.03)
+	)
+	(no_connect
+		(at 113.03 105.41)
+	)
+	(no_connect
+		(at 72.39 118.11)
+	)
+	(no_connect
+		(at 113.03 120.65)
+	)
+	(no_connect
+		(at 72.39 107.95)
+	)
+	(no_connect
+		(at 72.39 110.49)
+	)
+	(no_connect
+		(at 113.03 133.35)
+	)
+	(no_connect
+		(at 72.39 130.81)
+	)
 	(wire
 		(pts
@@
 	(wire
 		(pts
+			(xy 125.73 44.45) (xy 128.27 44.45)
+		)
+		(stroke
+			(width 0)
+			(type default)
+		)
+	)
+	(wire
+		(pts
 			(xy 119.38 128.27) (xy 119.38 129.54)
 		)
@@
 	(wire
 		(pts
+			(xy 172.72 116.84) (xy 175.26 116.84)
+		)
+		(stroke
+			(width 0)
+			(type default)
+		)
+	)
+	(wire
+		(pts
 			(xy 72.39 133.35) (xy 67.31 133.35)
 		)
@@
 	(wire
 		(pts
-			(xy 182.88 116.84) (xy 186.69 116.84)
-		)
-		(stroke
-			(width 0)
-			(type default)
-		)
-	)
-	(wire
-		(pts
 			(xy 113.03 135.89) (xy 119.38 135.89)
 		)
@@
 		(pts
 			(xy 123.19 46.99) (xy 125.73 46.99)
+		)
+		(stroke
+			(width 0)
+			(type default)
+		)
+	)
+	(wire
+		(pts
+			(xy 125.73 46.99) (xy 128.27 46.99)
 		)
 		(stroke
@@
 	)
 	(label "brightness"
-		(at 186.69 116.84 0)
+		(at 172.72 116.84 180)
 		(effects
 			(font
 				(size 1.27 1.27)
 			)
-			(justify left bottom)
+			(justify right bottom)
 		)
 	)
@@
 	)
 	(symbol
+		(lib_id "power:PWR_FLAG")
+		(at 128.27 44.45 270)
+		(unit 1)
+		(exclude_from_sim no)
+		(in_bom yes)
+		(on_board yes)
+		(dnp no)
+		(fields_autoplaced yes)
+		(property "Reference" "#FLG01"
+			(at 130.175 44.45 0)
+			(effects
+				(font
+					(size 1.27 1.27)
+				)
+				(hide yes)
+			)
+		)
+		(property "Value" "PWR_FLAG"
+			(at 132.08 44.4499 90)
+			(effects
+				(font
+					(size 1.27 1.27)
+				)
+				(justify left)
+			)
+		)
+		(property "Footprint" ""
+			(at 128.27 44.45 0)
+			(effects
+				(font
+					(size 1.27 1.27)
+				)
+				(hide yes)
+			)
+		)
+		(property "Datasheet" "~"
+			(at 128.27 44.45 0)
+			(effects
+				(font
+					(size 1.27 1.27)
+				)
+				(hide yes)
+			)
+		)
+		(property "Description" "Special symbol for telling ERC where power comes from"
+			(at 128.27 44.45 0)
+			(effects
+				(font
+					(size 1.27 1.27)
+				)
+				(hide yes)
+			)
+		)
+		(pin "1"
+		)
+		(instances
+			(project ""
+				(path "/390513d1-4e4f-4290-88d1-91fcabde20f5"
+					(reference "#FLG01")
+					(unit 1)
+				)
+			)
+		)
+	)
+	(symbol
 		(lib_id "Mechanical:MountingHole_Pad")
 		(at 219.71 54.61 0)
@@
 	(symbol
 		(lib_id "Device:R_Potentiometer")
-		(at 179.07 116.84 0)
+		(at 179.07 116.84 180)
 		(unit 1)
 		(exclude_from_sim no)
@@
 		(fields_autoplaced yes)
 		(property "Reference" "RV1"
-			(at 176.53 115.5699 0)
+			(at 181.61 115.5699 0)
 			(effects
 				(font
@@
 		)
 		(property "Value" "brightness_Pot"
-			(at 176.53 118.1099 0)
+			(at 181.61 118.1099 0)
 			(effects
 				(font
@@
 			)
 		)
-		(property "Footprint" ""
+		(property "Footprint" "Connector_PinHeader_2.54mm:PinHeader_1x03_P2.54mm_Vertical"
 			(at 179.07 116.84 0)
 			(effects
@@
 			)
 		)
-		(property "Footprint" ""
+		(property "Footprint" "Connector_PinHeader_2.54mm:PinHeader_1x02_P2.54mm_Vertical"
 			(at 209.55 116.84 0)
 			(effects
@@
 	)
 	(symbol
+		(lib_id "power:PWR_FLAG")
+		(at 128.27 46.99 270)
+		(unit 1)
+		(exclude_from_sim no)
+		(in_bom yes)
+		(on_board yes)
+		(dnp no)
+		(fields_autoplaced yes)
+		(property "Reference" "#FLG02"
+			(at 130.175 46.99 0)
+			(effects
+				(font
+					(size 1.27 1.27)
+				)
+				(hide yes)
+			)
+		)
+		(property "Value" "PWR_FLAG"
+			(at 132.08 46.9899 90)
+			(effects
+				(font
+					(size 1.27 1.27)
+				)
+				(justify left)
+			)
+		)
+		(property "Footprint" ""
+			(at 128.27 46.99 0)
+			(effects
+				(font
+					(size 1.27 1.27)
+				)
+				(hide yes)
+			)
+		)
+		(property "Datasheet" "~"
+			(at 128.27 46.99 0)
+			(effects
+				(font
+					(size 1.27 1.27)
+				)
+				(hide yes)
+			)
+		)
+		(property "Description" "Special symbol for telling ERC where power comes from"
+			(at 128.27 46.99 0)
+			(effects
+				(font
+					(size 1.27 1.27)
+				)
+				(hide yes)
+			)
+		)
+		(pin "1"
+		)
+		(instances
+			(project "logic"
+				(path "/390513d1-4e4f-4290-88d1-91fcabde20f5"
+					(reference "#FLG02")
+					(unit 1)
+				)
+			)
+		)
+	)
+	(symbol
 		(lib_id "Connector_Generic:Conn_01x02")
 		(at 118.11 46.99 180)
@@
 			)
 		)
-		(property "Value" "R"
+		(property "Value" "10k"
 			(at 217.17 132.0799 0)
 			(effects
@@
 			)
 		)
-		(property "Footprint" ""
+		(property "Footprint" "Resistor_THT:R_Axial_DIN0207_L6.3mm_D2.5mm_P10.16mm_Horizontal"
 			(at 212.852 130.81 90)
 			(effects
